File: Alturo/Proyecto kiss/Proyecto kiss.kicad_sch (KiCad schematic)
At the start: 9 parts, among them J1 TB3, J4 TB2

Commit message: Update Proyecto kiss.kicad_sch
Parts:
- added D1: Green_Led, LED_SMD:LED_1206_3216Metric, symbol Device:LED
- added R1: 220, Resistor_SMD:R_0201_0603Metric, symbol Device:R_Small_US
Connections:
- net Mod_Relay/12v_in is gone; now on net +12V: J4.2 (Pin_2)
- net Earth: now also D1.1 (K)
- new net: D1.2 (A), R1.2
- new net Mod_ESP32/Db_led: R1.1
Other:
- sheet Mod_ESP32 ports: added Db_led; removed none
Changed lines of the file:
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@@
   (junction (at 44.45 63.5) (diameter 0) (color 0 0 0 0)
   )
+  (junction (at 213.36 60.96) (diameter 0) (color 0 0 0 0)
+  )
   (junction (at 120.65 121.92) (diameter 0) (color 0 0 0 0)
   )
@@
     (stroke (width 0) (type default))
   )
+  (wire (pts (xy 213.36 60.96) (xy 213.36 67.31))
+    (stroke (width 0) (type default))
+  )
   (wire (pts (xy 114.3 135.89) (xy 118.11 135.89))
     (stroke (width 0) (type default))
@@
     (stroke (width 0) (type default))
   )
+  (wire (pts (xy 73.66 133.35) (xy 76.2 133.35))
+    (stroke (width 0) (type default))
+  )
   (wire (pts (xy 120.65 118.11) (xy 120.65 121.92))
     (stroke (width 0) (type default))
   )
+  (wire (pts (xy 76.2 140.97) (xy 76.2 143.51))
+    (stroke (width 0) (type default))
+  )
   (wire (pts (xy 44.45 69.85) (xy 44.45 66.04))
     (stroke (width 0) (type default))
@@
     (stroke (width 0) (type default))
   )
-  (wire (pts (xy 213.36 55.88) (xy 213.36 67.31))
+  (wire (pts (xy 213.36 55.88) (xy 213.36 60.96))
     (stroke (width 0) (type default))
   )
@@
   )
   (wire (pts (xy 33.02 111.76) (xy 36.83 111.76))
+    (stroke (width 0) (type default))
+  )
+  (wire (pts (xy 67.31 133.35) (xy 68.58 133.35))
     (stroke (width 0) (type default))
   )
@@
     )
   )
+  (symbol (lib_id "power:+12V") (at 213.36 60.96 90) (unit 1)
+    (in_bom yes) (on_board yes) (dnp no) (fields_autoplaced)
+    (property "Reference" "#PWR032" (at 217.17 60.96 0)
+      (effects (font (size 1.27 1.27)) hide)
+    )
+    (property "Value" "+12V" (at 209.55 61.595 90)
+      (effects (font (size 1.27 1.27)) (justify left))
+    )
+    (property "Footprint" "" (at 213.36 60.96 0)
+      (effects (font (size 1.27 1.27)) hide)
+    )
+    (property "Datasheet" "" (at 213.36 60.96 0)
+      (effects (font (size 1.27 1.27)) hide)
+    )
+    (pin "1")
+    (instances
+      (project "Proyecto kiss"
+        (path "/e9fd9658-b200-4aa5-b329-c1636df53c02"
+          (reference "#PWR032") (unit 1)
+        )
+      )
+    )
+  )
   (symbol (lib_id "power:+5V") (at 69.85 60.96 0) (unit 1)
     (in_bom yes) (on_board yes) (dnp no) (fields_autoplaced)
@@
     )
   )
+  (symbol (lib_id "Device:LED") (at 76.2 137.16 90) (unit 1)
+    (in_bom yes) (on_board yes) (dnp no)
+    (property "Reference" "D1" (at 78.74 135.89 90)
+      (effects (font (size 1.27 1.27)) (justify right))
+    )
+    (property "Value" "Green_Led" (at 78.74 138.43 90)
+      (effects (font (size 1.27 1.27)) (justify right) hide)
+    )
+    (property "Footprint" "LED_SMD:LED_1206_3216Metric" (at 76.2 137.16 0)
+      (effects (font (size 1.27 1.27)) hide)
+    )
+    (property "Datasheet" "https://www.rohm.com/datasheet?p=SML-S13PT&dist=Mouser&media=referral&source=mouser.com&campaign=Mouser" (at 76.2 137.16 0)
+      (effects (font (size 1.27 1.27)) hide)
+    )
+    (property "Manufacturer_Part_Number" "SML-S13PTT68" (at 76.2 137.16 0)
+      (effects (font (size 1.27 1.27)) hide)
+    )
+    (property "Mouser Price/Stock" "https://www.mouser.com/ProductDetail/ROHM-Semiconductor/SML-S13PTT68?qs=4v%252BiZTmLVHF1CiFCK4FhNg%3D%3D" (at 76.2 137.16 0)
+      (effects (font (size 1.27 1.27)) hide)
+    )
+    (pin "1")
+    (pin "2")
+    (instances
+      (project "reguladores"
+        (path "/cd16bd41-4f89-4d10-8c64-65342f721594"
+          (reference "D1") (unit 1)
+        )
+      )
+      (project "Proyecto kiss"
+        (path "/e9fd9658-b200-4aa5-b329-c1636df53c02"
+          (reference "D19") (unit 1)
+        )
+        (path "/e9fd9658-b200-4aa5-b329-c1636df53c02/a4128fef-9c50-4b7d-ad05-2e314a3c8b69"
+          (reference "D2") (unit 1)
+        )
+      )
+    )
+  )
   (symbol (lib_id "power:Earth") (at 114.3 123.19 0) (unit 1)
     (in_bom yes) (on_board yes) (dnp no) (fields_autoplaced)
@@
         (path "/e9fd9658-b200-4aa5-b329-c1636df53c02"
           (reference "#PWR015") (unit 1)
+        )
+      )
+    )
+  )
+  (symbol (lib_id "Device:R_Small_US") (at 71.12 133.35 90) (unit 1)
+    (in_bom yes) (on_board yes) (dnp no)
+    (property "Reference" "R1" (at 71.12 132.08 90)
+      (effects (font (size 1.27 1.27)))
+    )
+    (property "Value" "220" (at 71.12 135.89 90)
+      (effects (font (size 1.27 1.27)))
+    )
+    (property "Footprint" "Resistor_SMD:R_0201_0603Metric" (at 71.12 133.35 0)
+      (effects (font (size 1.27 1.27)) hide)
+    )
+    (property "Datasheet" "https://www.mouser.com/datasheet/2/427/crcw0201e3-1761851.pdf" (at 71.12 133.35 0)
+      (effects (font (size 1.27 1.27)) hide)
+    )
+    (property "Manufacturer_Part_Number" "CRCW0201220KFKED" (at 71.12 133.35 0)
+      (effects (font (size 1.27 1.27)) hide)
+    )
+    (property "Mouser Price/Stock" "https://www.mouser.com/ProductDetail/Vishay-Dale/CRCW0201220KFKED?qs=NYScm%2FwlDDYNqmB%252BWqlp%252Bw%3D%3D" (at 71.12 133.35 0)
+      (effects (font (size 1.27 1.27)) hide)
+    )
+    (pin "1")
+    (pin "2")
+    (instances
+      (project "reguladores"
+        (path "/cd16bd41-4f89-4d10-8c64-65342f721594"
+          (reference "R1") (unit 1)
+        )
+      )
+      (project "Proyecto kiss"
+        (path "/e9fd9658-b200-4aa5-b329-c1636df53c02"
+          (reference "R22") (unit 1)
+        )
+        (path "/e9fd9658-b200-4aa5-b329-c1636df53c02/a4128fef-9c50-4b7d-ad05-2e314a3c8b69"
+          (reference "R1") (unit 1)
         )
       )
@@
         (path "/e9fd9658-b200-4aa5-b329-c1636df53c02"
           (reference "J1") (unit 1)
+        )
+      )
+    )
+  )
+  (symbol (lib_id "power:Earth") (at 76.2 143.51 0) (unit 1)
+    (in_bom yes) (on_board yes) (dnp no) (fields_autoplaced)
+    (property "Reference" "#PWR04" (at 76.2 149.86 0)
+      (effects (font (size 1.27 1.27)) hide)
+    )
+    (property "Value" "Earth" (at 76.2 147.32 0)
+      (effects (font (size 1.27 1.27)) hide)
+    )
+    (property "Footprint" "" (at 76.2 143.51 0)
+      (effects (font (size 1.27 1.27)) hide)
+    )
+    (property "Datasheet" "~" (at 76.2 143.51 0)
+      (effects (font (size 1.27 1.27)) hide)
+    )
+    (pin "1")
+    (instances
+      (project "KISS_V2"
+        (path "/65dfba5e-78e0-455d-92b3-d370168d98c5/4b3fec45-17f7-4493-b982-1ebc81656281"
+          (reference "#PWR04") (unit 1)
+        )
+      )
+      (project "Proyecto kiss"
+        (path "/e9fd9658-b200-4aa5-b329-c1636df53c02"
+          (reference "#PWR031") (unit 1)
         )
       )
@@
       (effects (font (size 1.27 1.27)) (justify left))
     )
-    (instances
+    (pin "Db_led" input (at 67.31 133.35 0)
+      (effects (font (size 1.27 1.27)) (justify right))
+    )
+    (instances
