File: Alturo/Proyecto kiss/Mod_MPU-6500.kicad_sch (KiCad schematic)
At the start: 4 parts, among them U7 MPU-6500

Commit message: Update Mod_MPU-6500.kicad_sch
Parts:
- added R2 (x3): 10k, Resistor_SMD:R_0603_1608Metric, symbol Device:R
Connections:
- net Earth: now also R2.2, R2.2, R2.2
- net Pin_MPU: now also R2.1
- net SCL: now also R2.1
- net SDA: now also R2.1
Other:
- moved on the sheet: C10
