File: Alturo/Proyecto kiss/Proyecto kiss.kicad_pcb (KiCad board)
At the start: 2 copper layers, 127 x 127 mm, 72 parts, among them J1 IN/DC 12v, J2 VAL/ Out, J3 Relay / Out, J4 Sensor externo, J5 12V-ext_in, K1 FINDER-40.31, Q1 BSP75N, Q2 BC817, U1 AMS1117-3.3, U2 AMS1117-5.0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

Commit message: Update Proyecto kiss.kicad_pcb
Parts:
- added D19: Green_Led, LED_SMD:LED_1206_3216Metric, F.Cu at (173.1, 43.7)
- added R22: 220, Resistor_SMD:R_0201_0603Metric, F.Cu at (171.5, 46.3)
- BZ1, U5: moved to B.Cu
- C12, C15: value 100nF -> 100nf
- C14: value 100μF -> 100nf
- D10, D11, D12, D13, D14, D9: value LED -> Blue_Led
- D15, D16, D17, D18: value LED -> Yellow_Led
- D2: value LED -> Green_Led
- D3, D4, D5, D6, D7, D8: value LED -> Red_Led
- J1: value IN/DC 12v -> TB2
- J2: value VAL/ Out -> TB2
- J3: value Relay / Out -> TB2; footprint TerminalBlock_MetzConnect:TerminalBlock_MetzConnect_Type011_RT05503HBWC_1x03_P5.00mm_Horizontal -> TerminalBlock_MetzConnect:TerminalBlock_MetzConnect_Type011_RT05502HBWC_1x02_P5.00mm_Horizontal
- J4: value Sensor externo -> TB3
- J5: value 12V-ext_in -> TB2; moved to B.Cu
- RV1, RV2: value 60K -> 20K
- moved C10 156.4 mm to (-23.9, 80.9)
- moved R19 156.4 mm to (-19.2, 80.7)
- moved RV1 156.4 mm to (-14.3, 82.7)
- moved C9 156.4 mm to (-14.7, 89.7)
- moved J4 156.4 mm to (-5.59, 79.0)
- moved C8 125.8 mm to (-21.6, 63.2)
- moved R20 125.8 mm to (-13.4, 63.4)
- moved C11 125.8 mm to (-8.89, 63.1)
- moved RV2 125.8 mm to (-18.3, 60.9)
- moved U3 88.3 mm to (132.1, 184.4)
- moved U6 86.3 mm to (116.1, 179.8)
- moved C12 80.8 mm to (215.2, 109.2)
- moved C13 80.8 mm to (215.2, 110.9)
- moved C14 80.8 mm to (211.5, 107.1)
- moved U7 80.8 mm to (211.4, 110.1)
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Connections:
- J3 pad 1: /Mod_Relay/NO -> /Mod_Relay/Com
- J3 pad 2: /Mod_Relay/NC -> /Mod_Relay/NO
- J5 pad 2: /Mod_Relay/12v_in -> +12V
- K1 pad A1: /Mod_Relay/12v_in -> +12V
- U5 pad 26: unconnected-(U5-IO4-Pad26) -> /Mod_ESP32/Db_led
Routing:
- net Earth: track 0.00 -> 106.3 mm
- net Net-(D15-K): track 92.3 -> 0.00 mm
- net +12V: track 0.00 -> 71.9 mm
- net /Pin_RL: track 60.8 -> 0.00 mm
- net Net-(D10-K): track 57.8 -> 0.00 mm
- net +3.3V: track 0.00 -> 38.3 mm
- net /Mod_Relay/12v_in: track 38.0 -> 0.00 mm
- net Net-(#FLG02-pwr): track 0.00 -> 33.7 mm
- net Net-(U5-IO17): track 26.8 -> 0.00 mm
- net Net-(U5-IO16): track 26.3 -> 0.00 mm
- net +5V: track 3.30 -> 25.5 mm
- net /Mod_Relay/NC: track 21.3 -> 0.00 mm
- net /Pin_trans: track 20.1 -> 0.00 mm
- net /ledR: track 19.6 -> 0.00 mm
- net /ledB: track 19.0 -> 0.00 mm
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- added copper zone on In1.Cu, net Earth
Other:
- copper layers 2 -> 4

Commit message: Update Proyecto kiss.kicad_pcb
Parts:
- moved RV2 141.1 mm to (115.8, 104.6), turned to 180 degrees
- moved R20 127.3 mm to (109.0, 98.3), turned to 0 degrees
- moved C11 124.6 mm to (109.3, 102.7), turned to 90 degrees
- moved C8 116.4 mm to (93.7, 79.1)
- moved C10 91.0 mm to (61.7, 111.7)
- moved R19 83.9 mm to (57.7, 114.3), turned to 180 degrees
- moved RV1 73.3 mm to (54.8, 107.0), turned to 0 degrees
- moved C9 70.1 mm to (54.3, 102.1), turned to 180 degrees
- moved J4 61.1 mm to (45.7, 112.2), turned to 90 degrees
Routing:
- net Earth: track 106.3 -> 159.7 mm
- net /Sen_ext: track 0.00 -> 27.6 mm
- net /Sen_int: track 0.00 -> 21.1 mm
- net Net-(J4-Pin_3): track 0.00 -> 7.88 mm

Commit message: Update Proyecto kiss.kicad_pcb
Parts:
- moved C13 103.2 mm to (117.1, 143.0), turned to -90 degrees
- moved C12 102.8 mm to (117.1, 139.9), turned to -90 degrees
- moved U7 102.6 mm to (114.0, 142.5)
- moved C14 101.9 mm to (114.8, 139.2)
Routing:
- net /SCL: track 0.00 -> 14.1 mm
- net Earth: track 159.7 -> 166.7 mm
- net Net-(U7-REGOUT): track 0.00 -> 4.05 mm
- net +3.3V: track 38.3 -> 42.0 mm
- net /SDA: track 0.00 -> 2.76 mm

Commit message: Update Proyecto kiss.kicad_pcb
Parts:
- moved U3 70.8 mm to (129.5, 113.7)
- moved U6 66.2 mm to (116.5, 113.7)
- moved C13 1.29 mm to (117.9, 144.0), turned to 180 degrees
- moved C12 1.27 mm to (117.8, 141.0), turned to 0 degrees
Routing:
- net /Pin_MPU: track 0.00 -> 49.5 mm
- net /ledR: track 0.00 -> 32.9 mm
- net /ledB: track 0.00 -> 31.5 mm
- net /ledY: track 0.00 -> 30.2 mm
- net Net-(U5-IO17): track 0.00 -> 16.0 mm
- net Net-(U5-IO16): track 0.00 -> 15.4 mm
- net Earth: track 166.7 -> 178.2 mm
- net Net-(U7-REGOUT): track 4.05 -> 2.34 mm

Commit message: Update Proyecto kiss.kicad_pcb
Parts:
- moved D19 138.2 mm to (81.3, 146.9), turned to 90 degrees
- moved R22 132.4 mm to (81.3, 143.2), turned to -90 degrees
- moved D14 91.6 mm to (150.4, 94.9), turned to 90 degrees
- moved D5 91.5 mm to (71.1, 49.3), turned to -150 degrees
- moved R5 81.3 mm to (77.5, 68.3), turned to 30 degrees
- moved R14 78.2 mm to (142.0, 90.2), turned to -90 degrees
- moved D13 69.7 mm to (137.7, 94.9), turned to 90 degrees
- moved D4 69.6 mm to (77.2, 60.5), turned to -150 degrees
- moved R4 66.3 mm to (79.5, 71.9), turned to 30 degrees
- moved R13 63.8 mm to (137.7, 90.2), turned to -90 degrees
- moved R3 48.9 mm to (81.5, 75.4), turned to 30 degrees
- moved R12 48.1 mm to (133.3, 90.2), turned to -90 degrees
- moved D12 43.4 mm to (122.4, 94.9), turned to 90 degrees
- moved D3 43.1 mm to (85.1, 73.4), turned to -150 degrees
- moved R8 24.2 mm to (117.9, 68.7)
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Routing:
- net +5V: track 25.5 -> 139.6 mm
- net Net-(D3-K): track 0.00 -> 82.3 mm
- net Net-(D15-K): track 0.00 -> 75.0 mm
- net /Mod_ESP32/Db_led: track 0.00 -> 61.9 mm
- net Net-(D10-K): track 0.00 -> 55.9 mm
- net +12V: track 71.9 -> 103.0 mm
- net Net-(D8-A): track 0.00 -> 21.6 mm
- net Net-(D5-A): track 0.00 -> 21.3 mm
- net Net-(D9-A): track 0.00 -> 14.2 mm
- net Net-(D7-A): track 0.00 -> 12.7 mm
- net Net-(D4-A): track 0.00 -> 12.1 mm
- net Net-(D12-A): track 0.00 -> 11.9 mm
- net Net-(D11-A): track 0.00 -> 11.6 mm
- net Net-(D15-A): track 0.00 -> 11.2 mm
- net Net-(D18-A): track 0.00 -> 10.4 mm
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
Commit message: Update Proyecto kiss.kicad_pcb
Parts:
- added R23: 10k, Resistor_SMD:R_0603_1608Metric, F.Cu at (113.3, 140.5)
- added R24: 10k, Resistor_SMD:R_0603_1608Metric, F.Cu at (113.3, 142.2)
- added R25: 10k, Resistor_SMD:R_0603_1608Metric, F.Cu at (114.8, 152.1)
- moved BZ1 66.6 mm to (131.3, 128.3)
- moved Q2 64.3 mm to (133.8, 136.7), turned to 0 degrees
- moved R21 59.5 mm to (130.1, 135.8), turned to 0 degrees
- moved C14 13.4 mm to (118.1, 152.1)
- moved C12 8.39 mm to (118.1, 149.4)
- moved C13 6.16 mm to (114.8, 149.4)
- moved U7 4.17 mm to (116.6, 145.8), turned to 0 degrees
- moved U6 1.07 mm to (117.6, 113.7), turned to 90 degrees
- moved D10 0.25 mm to (57.1, 94.9)
- moved D11 0.23 mm to (44.4, 94.9)
- moved D9 0.18 mm to (72.3, 94.9)
- turned U3 to 90 degrees
Connections:
- U3 pad 8: GNDREF -> Earth
Routing:
- net +5V: track 139.6 -> 307.7 mm, vias 0 -> 6
- net +3.3V: track 46.7 -> 160.0 mm, vias 0 -> 5
- net /Pin_trans: track 0.00 -> 82.2 mm, vias 0 -> 2
- net Net-(D10-K): track 55.9 -> 121.8 mm
- net /Sen_int: track 21.1 -> 75.0 mm
- net Net-(D3-K): track 82.3 -> 128.8 mm, vias 0 -> 2
- net Net-(D15-K): track 75.0 -> 118.3 mm
- net /Pin_RL: track 0.00 -> 40.9 mm, vias 0 -> 1
- net /Sen_ext: track 27.6 -> 67.7 mm, vias 0 -> 1
- net +12V: track 103.0 -> 136.6 mm, vias 0 -> 1
- net /Pin_bzz: track 0.00 -> 31.2 mm, vias 0 -> 1
- net /ledR: track 32.9 -> 53.8 mm
- net /ledB: track 31.5 -> 47.7 mm
- net Net-(U4-A1): track 7.85 -> 22.1 mm
- net /SDA: track 2.76 -> 10.4 mm, vias 0 -> 1
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
Commit message: Update Proyecto kiss.kicad_pcb
Parts:
- moved R3 9.12 mm to (72.6, 73.4), turned to 0 degrees
- moved R4 7.03 mm to (72.6, 70.4), turned to 0 degrees
- moved R8 5.63 mm to (121.6, 72.9), turned to 90 degrees
- moved R5 4.93 mm to (72.6, 67.3), turned to 0 degrees
- moved R6 3.71 mm to (116.1, 72.8), turned to 90 degrees
- moved R7 3.01 mm to (118.8, 72.8), turned to 90 degrees
- moved D1 1.27 mm to (115.8, 41.1)
- moved C15 0.51 mm to (81.3, 153.1)
- moved D2 0.34 mm to (91.6, 55.7)
- turned D15 to 180 degrees
- turned D16 to 180 degrees
- turned D17 to 0 degrees
- turned D18 to 0 degrees
- turned D3 to 180 degrees
- turned D4 to 180 degrees
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Routing:
- net +5V: track 307.7 -> 338.5 mm
- net Net-(D3-K): track 128.8 -> 153.6 mm
- net Net-(D15-K): track 118.3 -> 137.4 mm
- net Earth: track 180.5 -> 194.3 mm
- net /Pin_MPU: track 44.9 -> 57.4 mm
- net +3.3V: track 160.0 -> 171.4 mm
- net Net-(D3-A): track 2.01 -> 10.2 mm
- net /Sen_ext: track 67.7 -> 75.7 mm
- net /Mod_ESP32/Db_led: track 62.5 -> 69.2 mm
- net Net-(D8-A): track 21.6 -> 26.4 mm
- net +12V: track 136.6 -> 141.4 mm
- net /Sen_int: track 75.0 -> 79.6 mm
- net /Pin_bzz: track 31.2 -> 35.6 mm
- net Net-(D6-A): track 2.52 -> 6.05 mm
- net /ledR: track 53.8 -> 57.3 mm
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